File: hardware/TDSE-TF/TDSE-TF.kicad_pcb (KiCad board)
At the start: 2 copper layers, 149.9 x 89.9 mm, 48 parts, among them J1 Sensor agua, J10 CN10, J2 Tira LED, J3 +5VCC, J5 Bomba, J6 Sensor luz, J7 CN7, J8 Sensor humedad, J9 Conector LCD16x02, Q1 IRLZ44, Q2 IRLZ44, Q3 MPSA42, SW1 Enter, SW2 Anterior, SW3 Siguiente, SW4 Escape, U1 DHT22

Commit message: Update KiCad TDSE-TF PCB & schematic
Modify TDSE-TF KiCad project: add diode D4 (1N4007) and resistor R9 (axial) symbols/footprints; adjust resistor values/labels (e.g. 3R3, 56). Update PCB file: layer selection, mirror setting, pad sizes/drills, nets and routing (several Net-(J5-Pin_2) -> Net-(D4-A), Net-(Q1-G) and /Driver Bomba adjustments), silkscreen/fab text positions and many footprint placements. Update project metadata (.kicad_prl/.kicad_pro) including active layer, column widths and used_designators; bump board Rev to 7. Remove Measurements SMARTCETA.txt and add ~TDSE-TF.kicad_pro.lck lock file. Changes reflect placement/routing and part additions for the TDSE-TF hardware revision.
Parts:
- added D4: 1N4007, Diode_THT:D_DO-41_SOD81_P10.16mm_Horizontal, F.Cu at (221.9, 17.0)
- added R9: 56, Resistor_THT:R_Axial_DIN0207_L6.3mm_D2.5mm_P10.16mm_Horizontal, F.Cu at (260.9, 35.7)
- J1: value Sensor agua -> Nivel agua
- J6: value Sensor luz -> Nivel luz
- J8: value Sensor humedad -> Humedad sustrato
- R2: value TBD -> 3R3
Connections:
- Q1 pad 1: /Driver Bomba -> Net-(Q1-G)
Routing:
- net /Driver Bomba: track 89.3 -> 70.2 mm
- net Net-(Q1-G): track 0.00 -> 10.5 mm
- net Net-(D4-A): track 65.5 -> 74.8 mm
Other:
- board text added: "Rev 7"
- board text removed: "Rev 6"
