File: hardware/TDSE-TF/TDSE-TF.kicad_sch (KiCad schematic)
At the start: 30 parts, among them J1 Sensor nivel de agua, J10 CN10, J2 Tira LED, J3 +5VCC entrada, J5 Bomba, J6 Sensor nivel de luz, J7 CN7, J8 Sensor humedad de suelo, J9 Conector LCD16x02, Q1 IRLZ44, Q2 IRLZ44, Q3 MPSA42, SW1 Enter, SW2 Anterior, SW3 Siguiente, SW4 Escape, U1 DHT22

Commit message: Update KiCad TDSE-TF PCB & schematic
Modify TDSE-TF KiCad project: add diode D4 (1N4007) and resistor R9 (axial) symbols/footprints; adjust resistor values/labels (e.g. 3R3, 56). Update PCB file: layer selection, mirror setting, pad sizes/drills, nets and routing (several Net-(J5-Pin_2) -> Net-(D4-A), Net-(Q1-G) and /Driver Bomba adjustments), silkscreen/fab text positions and many footprint placements. Update project metadata (.kicad_prl/.kicad_pro) including active layer, column widths and used_designators; bump board Rev to 7. Remove Measurements SMARTCETA.txt and add ~TDSE-TF.kicad_pro.lck lock file. Changes reflect placement/routing and part additions for the TDSE-TF hardware revision.
Parts:
- added D4: 1N4007, Diode_THT:D_DO-41_SOD81_P10.16mm_Horizontal, symbol Diode:1N4007
- added R9: 56, Resistor_THT:R_Axial_DIN0207_L6.3mm_D2.5mm_P10.16mm_Horizontal, symbol Device:R
- R2: value TBD -> 3R3
Connections:
- net Driver Bomba: now also R9.1; no longer Q1.1 (G)
- net VCC: now also D4.1 (K)
- net at J5.2 (Pin_2), Q1.2 (D): now also D4.2 (A)
- new net: Q1.1 (G), R9.2
